Commit message: Gazebo file okay

File: max_description/urdf/materials.xacro (robot description, xacro)
@@ -1,6 +1,15 @@
 <?xml version="1.0" ?>
 <robot name="max" xmlns:xacro="http://www.ros.org/wiki/xacro" >
+    <!-- Base body -->
     <material name="silver">
-    <color rgba="0.700 0.700 0.700 1.000"/>
+        <color rgba="0.700 0.700 0.700 1.000"/>
+    </material>
+    <!-- Wheels -->
+    <material name="matte_black">
+        <color rgba="0.05 0.05 0.05 1.0"/>
+    </material>
+    <!-- Lidar -->
+    <material name="tech_blue">
+        <color rgba="0.0 0.3 0.6 1.0"/>
     </material>
 </robot>

File: max_description/urdf/max.urdf.xacro (robot description, xacro)
@@ -35,5 +35,5 @@
                 <mesh filename="file://$(find max_description)/meshes/fl_wheel_link.stl" scale="0.001 0.001 0.001"/>
             </geometry>
-            <material name="silver"/>
+            <material name="matte_black"/>
         </visual>
         <collision>
@@ -55,5 +55,5 @@
             <mesh filename="file://$(find max_description)/meshes/fr_wheel_link.stl" scale="0.001 0.001 0.001"/>
             </geometry>
-            <material name="silver"/>
+            <material name="matte_black"/>
         </visual>
         <collision>
@@ -75,5 +75,5 @@
             <mesh filename="file://$(find max_description)/meshes/rl_wheel_link.stl" scale="0.001 0.001 0.001"/>
             </geometry>
-            <material name="silver"/>
+            <material name="matte_black"/>
         </visual>
         <collision>
@@ -95,5 +95,5 @@
             <mesh filename="file://$(find max_description)/meshes/rr_wheel_link.stl" scale="0.001 0.001 0.001"/>
             </geometry>
-            <material name="silver"/>
+            <material name="matte_black"/>
         </visual>
         <collision>
@@ -115,5 +115,5 @@
             <mesh filename="file://$(find max_description)/meshes/lidar_link.stl" scale="0.001 0.001 0.001"/>
             </geometry>
-            <material name="silver"/>
+            <material name="tech_blue"/>
         </visual>
         <collision>

Commit message: added camera lnk to urdf

File: max_description/urdf/materials.xacro (robot description, xacro)
@@ -13,3 +13,7 @@
         <color rgba="0.0 0.3 0.6 1.0"/>
     </material>
+    <!-- Camera -->
+    <material name="camera_accent">
+        <color rgba="0.0 0.5 1.0 1.0"/>
+    </material>
 </robot>

File: max_description/urdf/max.gazebo.xacro (robot description, xacro)
@@ -3,4 +3,5 @@
   <xacro:property name="wheel_color" value="Gazebo/Black" />
   <xacro:property name="lidar_color" value="Gazebo/Blue" />
+  <xacro:property name="camera_color" value="Gazebo/Grey" />
   <gazebo reference="fl_wheel_link">
     <material>${wheel_color}</material>
@@ -46,3 +47,6 @@
     <material>${lidar_color}</material>
   </gazebo>
+  <gazebo reference="camera_link_1">
+    <material>${camera_color}</material>
+  </gazebo>
 </robot>

File: max_description/urdf/max.urdf.xacro (robot description, xacro)
@@ -124,4 +124,24 @@
         </collision>
     </link>
+    <link name="camera_link">
+        <inertial>
+            <origin xyz="0.014490312898766358 3.7392359944188856e-16 -0.008993541932510896" rpy="0 0 0"/>
+            <mass value="1.7184205751165316"/>
+            <inertia ixx="0.00474" iyy="0.000448" izz="0.004472" ixy="0.0" iyz="-0.0" ixz="0.0"/>
+        </inertial>
+        <visual>
+            <origin xyz="-0.1133 -0.0 -0.144" rpy="0 0 0"/>
+            <geometry>
+            <mesh filename="file://$(find max_description)/meshes/camera_link.stl" scale="0.001 0.001 0.001"/>
+            </geometry>
+            <material name="camera_accent"/>
+        </visual>
+        <collision>
+            <origin xyz="-0.1133 -0.0 -0.144" rpy="0 0 0"/>
+            <geometry>
+            <mesh filename="file://$(find max_description)/meshes/camera_link.stl" scale="0.001 0.001 0.001"/>
+            </geometry>
+        </collision>
+    </link>
     <joint name="base_joint" type="fixed">
         <parent link="base_footprint"/>
@@ -159,3 +179,8 @@
         <axis xyz="0 0 1"/>
     </joint>
+    <joint name="camera_joint" type="fixed">
+        <origin xyz="0.1133 0.0 0.1015" rpy="0 0 0"/>
+        <parent link="base_link"/>
+        <child link="camera_link"/>
+    </joint>
 </robot>
