Commit message: Fixed gazebo sinking max

File: max_description/urdf/max.gazebo.xacro (robot description, xacro)
@@ -1,39 +1,44 @@
 <?xml version="1.0" ?>
 <robot name="max" xmlns:xacro="http://www.ros.org/wiki/xacro" >
+  <xacro:property name="body_color" value="Gazebo/Silver" />
+  <gazebo>
+    <plugin name="control" filename="libgazebo_ros_control.so"/>
+  </gazebo>
+  <gazebo reference="base_link">
+    <material>${body_color}</material>
+    <mu1>0.2</mu1>
+    <mu2>0.2</mu2>
+    <self_collide>true</self_collide>
+    <gravity>true</gravity>
+  </gazebo>
   <gazebo reference="fl_wheel_link">
-    <mu1>100000000000000.0</mu1>
-    <mu2>100000000000000.0</mu2>
-    <kp>1000000000000.0</kp>
-    <kd>10.0</kd>
-    <minDepth>0.001</minDepth>
-    <maxVel>0.1</maxVel>
-    <fdir1>1 0 0</fdir1>
+    <material>${body_color}</material>
+    <mu1>0.2</mu1>
+    <mu2>0.2</mu2>
+    <self_collide>true</self_collide>
   </gazebo>
   <gazebo reference="fr_wheel_link">
-    <mu1>100000000000000.0</mu1>
-    <mu2>100000000000000.0</mu2>
-    <kp>1000000000000.0</kp>
-    <kd>10.0</kd>
-    <minDepth>0.001</minDepth>
-    <maxVel>0.1</maxVel>
-    <fdir1>1 0 0</fdir1>
+    <material>${body_color}</material>
+    <mu1>0.2</mu1>
+    <mu2>0.2</mu2>
+    <self_collide>true</self_collide>
   </gazebo>
   <gazebo reference="rl_wheel_link">
-    <mu1>100000000000000.0</mu1>
-    <mu2>100000000000000.0</mu2>
-    <kp>1000000000000.0</kp>
-    <kd>10.0</kd>
-    <minDepth>0.001</minDepth>
-    <maxVel>0.1</maxVel>
-    <fdir1>1 0 0</fdir1>
+    <material>${body_color}</material>
+    <mu1>0.2</mu1>
+    <mu2>0.2</mu2>
+    <self_collide>true</self_collide>
   </gazebo>
   <gazebo reference="rr_wheel_link">
-    <mu1>100000000000000.0</mu1>
-    <mu2>100000000000000.0</mu2>
-    <kp>1000000000000.0</kp>
-    <kd>10.0</kd>
-    <minDepth>0.001</minDepth>
-    <maxVel>0.1</maxVel>
-    <fdir1>1 0 0</fdir1>
+    <material>${body_color}</material>
+    <mu1>0.2</mu1>
+    <mu2>0.2</mu2>
+    <self_collide>true</self_collide>
+  </gazebo>
+  <gazebo reference="lidar_link">
+    <material>${body_color}</material>
+    <mu1>0.2</mu1>
+    <mu2>0.2</mu2>
+    <self_collide>true</self_collide>
   </gazebo>
 </robot>

File: max_description/urdf/max.urdf.xacro (robot description, xacro)
@@ -40,5 +40,5 @@
             <origin xyz="-0.07309 -0.109 -0.0425" rpy="0 0 0"/>
             <geometry>
-                <sphere radius="0.0425"/>
+            <mesh filename="file://$(find max_description)/meshes/fl_wheel_link.stl" scale="0.001 0.001 0.001"/>
             </geometry>
         </collision>
@@ -60,5 +60,5 @@
             <origin xyz="-0.07309 0.109 -0.0425" rpy="0 0 0"/>
             <geometry>
-                <sphere radius="0.0425"/>
+            <mesh filename="file://$(find max_description)/meshes/fr_wheel_link.stl" scale="0.001 0.001 0.001"/>
             </geometry>
         </collision>
@@ -80,5 +80,5 @@
             <origin xyz="0.0978 -0.109 -0.0425" rpy="0 0 0"/>
             <geometry>
-                <sphere radius="0.0425"/>
+            <mesh filename="file://$(find max_description)/meshes/rl_wheel_link.stl" scale="0.001 0.001 0.001"/>
             </geometry>
         </collision>
@@ -100,5 +100,5 @@
             <origin xyz="0.0978 0.109 -0.0425" rpy="0 0 0"/>
             <geometry>
-                <sphere radius="0.0425"/>
+            <mesh filename="file://$(find max_description)/meshes/rr_wheel_link.stl" scale="0.001 0.001 0.001"/>
             </geometry>
         </collision>
@@ -119,4 +119,7 @@
         <collision>
             <origin xyz="-0.0 -0.0 -0.204001" rpy="0 0 0"/>
+            <geometry>
+            <mesh filename="file://$(find max_description)/meshes/lidar_link.stl" scale="0.001 0.001 0.001"/>
+            </geometry>
         </collision>
     </link>

Commit message: Gazebo file okay

File: max_description/urdf/max.gazebo.xacro (robot description, xacro)
@@ -1,44 +1,48 @@
 <?xml version="1.0" ?>
 <robot name="max" xmlns:xacro="http://www.ros.org/wiki/xacro" >
-  <xacro:property name="body_color" value="Gazebo/Silver" />
-  <gazebo>
-    <plugin name="control" filename="libgazebo_ros_control.so"/>
-  </gazebo>
-  <gazebo reference="base_link">
-    <material>${body_color}</material>
-    <mu1>0.2</mu1>
-    <mu2>0.2</mu2>
-    <self_collide>true</self_collide>
-    <gravity>true</gravity>
-  </gazebo>
+  <xacro:property name="wheel_color" value="Gazebo/Black" />
+  <xacro:property name="lidar_color" value="Gazebo/Blue" />
   <gazebo reference="fl_wheel_link">
-    <material>${body_color}</material>
-    <mu1>0.2</mu1>
-    <mu2>0.2</mu2>
-    <self_collide>true</self_collide>
+    <material>${wheel_color}</material>
+    <mu1>1.0</mu1>
+    <mu2>1.0</mu2>
+    <kp>100000.0</kp>
+    <kd>5.0</kd>
+    <minDepth>0.001</minDepth>
+    <maxVel>0.2</maxVel>
+    <fdir1>1 0 0</fdir1>
   </gazebo>
   <gazebo reference="fr_wheel_link">
-    <material>${body_color}</material>
-    <mu1>0.2</mu1>
-    <mu2>0.2</mu2>
-    <self_collide>true</self_collide>
+    <material>${wheel_color}</material>
+    <mu1>1.0</mu1>
+    <mu2>1.0</mu2>
+    <kp>100000.0</kp>
+    <kd>5.0</kd>
+    <minDepth>0.001</minDepth>
+    <maxVel>0.2</maxVel>
+    <fdir1>1 0 0</fdir1>
   </gazebo>
   <gazebo reference="rl_wheel_link">
-    <material>${body_color}</material>
-    <mu1>0.2</mu1>
-    <mu2>0.2</mu2>
-    <self_collide>true</self_collide>
+    <material>${wheel_color}</material>
+    <mu1>1.0</mu1>
+    <mu2>1.0</mu2>
+    <kp>100000.0</kp>
+    <kd>5.0</kd>
+    <minDepth>0.001</minDepth>
+    <maxVel>0.2</maxVel>
+    <fdir1>1 0 0</fdir1>
   </gazebo>
   <gazebo reference="rr_wheel_link">
-    <material>${body_color}</material>
-    <mu1>0.2</mu1>
-    <mu2>0.2</mu2>
-    <self_collide>true</self_collide>
+    <material>${wheel_color}</material>
+    <mu1>1.0</mu1>
+    <mu2>1.0</mu2>
+    <kp>100000.0</kp>
+    <kd>5.0</kd>
+    <minDepth>0.001</minDepth>
+    <maxVel>0.2</maxVel>
+    <fdir1>1 0 0</fdir1>
   </gazebo>
   <gazebo reference="lidar_link">
-    <material>${body_color}</material>
-    <mu1>0.2</mu1>
-    <mu2>0.2</mu2>
-    <self_collide>true</self_collide>
+    <material>${lidar_color}</material>
   </gazebo>
 </robot>

Commit message: added camera lnk to urdf

File: max_description/urdf/max.gazebo.xacro (robot description, xacro)
@@ -3,5 +3,5 @@
   <xacro:property name="wheel_color" value="Gazebo/Black" />
   <xacro:property name="lidar_color" value="Gazebo/Blue" />
-  <xacro:property name="camera_color" value="Gazebo/Grey" />
+  <xacro:property name="camera_color" value="Gazebo/Blue" />
   <gazebo reference="fl_wheel_link">
     <material>${wheel_color}</material>
@@ -47,5 +47,5 @@
     <material>${lidar_color}</material>
   </gazebo>
-  <gazebo reference="camera_link_1">
+  <gazebo reference="camera_link">
     <material>${camera_color}</material>
   </gazebo>

Commit message: Beginning on diff drive controller

File: max_description/urdf/max.gazebo.xacro (robot description, xacro)
@@ -4,23 +4,13 @@
   <xacro:property name="lidar_color" value="Gazebo/Blue" />
   <xacro:property name="camera_color" value="Gazebo/Blue" />
-  <gazebo reference="fl_wheel_link">
+  <gazebo reference="fr_roller_wheel">
     <material>${wheel_color}</material>
-    <mu1>1.5</mu1>
-    <mu2>0.5</mu2>
-    <kp>100000.0</kp>
-    <kd>10.0</kd>
-    <minDepth>0.001</minDepth>
-    <maxVel>0.5</maxVel>
-    <fdir1>1 0 0</fdir1>
+    <mu1>0.2</mu1>
+    <mu2>0.2</mu2>
   </gazebo>
-  <gazebo reference="fr_wheel_link">
+  <gazebo reference="fl_roller_wheel">
     <material>${wheel_color}</material>
-    <mu1>1.5</mu1>
-    <mu2>0.5</mu2>
-    <kp>100000.0</kp>
-    <kd>10.0</kd>
-    <minDepth>0.001</minDepth>
-    <maxVel>0.5</maxVel>
-    <fdir1>1 0 0</fdir1>
+    <mu1>0.2</mu1>
+    <mu2>0.2</mu2>
   </gazebo>
   <gazebo reference="rl_wheel_link">

File: max_description/urdf/max.urdf.xacro (robot description, xacro)
@@ -10,7 +10,7 @@
     <link name="base_link">
         <inertial>
-            <origin xyz="0.004914987095310725 0.0 0.11525864563546669" rpy="0 0 0"/>
-            <mass value="2.1411582458682883"/>
-            <inertia ixx="0.015376" iyy="0.021164" izz="0.024064" ixy="-0.0" iyz="-0.0" ixz="0.000293"/>
+            <origin xyz="-0.02395632727900399 -2.01772150977478e-07 0.09083712403458968" rpy="0 0 0"/>
+            <mass value="2.2280671864878805"/>
+            <inertia ixx="0.010988" iyy="0.012735" izz="0.013502" ixy="0.0" iyz="0.0" ixz="0.0016"/>
         </inertial>
         <visual>
@@ -24,45 +24,25 @@
             <origin xyz="0 0 0" rpy="0 0 0"/>
             <geometry>
-                <mesh filename="file://$(find max_description)/meshes/base_link.stl" scale="0.001 0.001 0.001"/>
+            <mesh filename="file://$(find max_description)/meshes/base_link.stl" scale="0.001 0.001 0.001"/>
             </geometry>
         </collision>
     </link>
-    <link name="fl_wheel_link">
+    <link name="rr_wheel_link">
         <inertial>
-            <origin xyz="4.163336342344337e-17 0.010504987657416559 -1.3877787807814457e-17" rpy="0 0 0"/>
-            <mass value="0.15230338417321157"/>
-            <inertia ixx="8.3e-05" iyy="0.000141" izz="8.3e-05" ixy="0.0" iyz="-0.0" ixz="-0.0"/>
+            <origin xyz="-2.2343238370581275e-15 -0.015512778351276846 1.3877787807814457e-17" rpy="0 0 0"/>
+            <mass value="0.14404511942595016"/>
+            <inertia ixx="8.7e-05" iyy="0.000137" izz="8.7e-05" ixy="0.0" iyz="0.0" ixz="0.0"/>
         </inertial>
         <visual>
-            <origin xyz="-0.07309 -0.109 -0.0425" rpy="0 0 0"/>
+            <origin xyz="0.075 0.095 -0.0425" rpy="0 0 0"/>
             <geometry>
-                <mesh filename="file://$(find max_description)/meshes/fl_wheel_link.stl" scale="0.001 0.001 0.001"/>
+            <mesh filename="file://$(find max_description)/meshes/rr_wheel_link.stl" scale="0.001 0.001 0.001"/>
             </geometry>
             <material name="matte_black"/>
         </visual>
         <collision>
-            <origin xyz="-0.07309 -0.109 -0.0425" rpy="0 0 0"/>
+            <origin xyz="0.075 0.095 -0.0425" rpy="0 0 0"/>
             <geometry>
-            <mesh filename="file://$(find max_description)/meshes/fl_wheel_link.stl" scale="0.001 0.001 0.001"/>
-            </geometry>
-        </collision>
-    </link>
-    <link name="fr_wheel_link">
-        <inertial>
-            <origin xyz="4.163336342344337e-17 -0.010504987657416545 -1.3877787807814457e-17" rpy="0 0 0"/>
-            <mass value="0.15230338417321157"/>
-            <inertia ixx="8.3e-05" iyy="0.000141" izz="8.3e-05" ixy="0.0" iyz="0.0" ixz="-0.0"/>
-        </inertial>
-        <visual>
-            <origin xyz="-0.07309 0.109 -0.0425" rpy="0 0 0"/>
-            <geometry>
-            <mesh filename="file://$(find max_description)/meshes/fr_wheel_link.stl" scale="0.001 0.001 0.001"/>
-            </geometry>
-            <material name="matte_black"/>
-        </visual>
-        <collision>
-            <origin xyz="-0.07309 0.109 -0.0425" rpy="0 0 0"/>
-            <geometry>
-            <mesh filename="file://$(find max_description)/meshes/fr_wheel_link.stl" scale="0.001 0.001 0.001"/>
+            <mesh filename="file://$(find max_description)/meshes/rr_wheel_link.stl" scale="0.001 0.001 0.001"/>
             </geometry>
         </collision>
@@ -70,10 +50,10 @@
     <link name="rl_wheel_link">
         <inertial>
-            <origin xyz="6.938893903907228e-17 0.010504987657416559 0.0" rpy="0 0 0"/>
-            <mass value="0.15230338417321163"/>
-            <inertia ixx="8.3e-05" iyy="0.000141" izz="8.3e-05" ixy="0.0" iyz="-0.0" ixz="0.0"/>
+            <origin xyz="-2.220446049250313e-16 0.015512778351276832 6.245004513516506e-17" rpy="0 0 0"/>
+            <mass value="0.1440451194259502"/>
+            <inertia ixx="8.7e-05" iyy="0.000137" izz="8.7e-05" ixy="-0.0" iyz="0.0" ixz="0.0"/>
         </inertial>
         <visual>
-            <origin xyz="0.0978 -0.109 -0.0425" rpy="0 0 0"/>
+            <origin xyz="0.075 -0.095 -0.0425" rpy="0 0 0"/>
             <geometry>
             <mesh filename="file://$(find max_description)/meshes/rl_wheel_link.stl" scale="0.001 0.001 0.001"/>
@@ -82,5 +62,5 @@
         </visual>
         <collision>
-            <origin xyz="0.0978 -0.109 -0.0425" rpy="0 0 0"/>
+            <origin xyz="0.075 -0.095 -0.0425" rpy="0 0 0"/>
             <geometry>
             <mesh filename="file://$(find max_description)/meshes/rl_wheel_link.stl" scale="0.001 0.001 0.001"/>
@@ -88,32 +68,12 @@
         </collision>
     </link>
-    <link name="rr_wheel_link">
+    <link name="lidar_link">
         <inertial>
-            <origin xyz="6.938893903907228e-17 -0.010504987657416559 -2.0816681711721685e-17" rpy="0 0 0"/>
-            <mass value="0.15230338417321163"/>
-            <inertia ixx="8.3e-05" iyy="0.000141" izz="8.3e-05" ixy="-0.0" iyz="0.0" ixz="0.0"/>
+            <origin xyz="-6.154361288395009e-18 -4.3080529018765064e-17 0.012000000000000038" rpy="0 0 0"/>
+            <mass value="0.09790459345647239"/>
+            <inertia ixx="3.5e-05" iyy="3.5e-05" izz="6e-05" ixy="0.0" iyz="0.0" ixz="0.0"/>
         </inertial>
         <visual>
-            <origin xyz="0.0978 0.109 -0.0425" rpy="0 0 0"/>
-            <geometry>
-            <mesh filename="file://$(find max_description)/meshes/rr_wheel_link.stl" scale="0.001 0.001 0.001"/>
-            </geometry>
-            <material name="matte_black"/>
-        </visual>
-        <collision>
-            <origin xyz="0.0978 0.109 -0.0425" rpy="0 0 0"/>
-            <geometry>
-            <mesh filename="file://$(find max_description)/meshes/rr_wheel_link.stl" scale="0.001 0.001 0.001"/>
-            </geometry>
-        </collision>
-    </link>
-    <link name="lidar_link">
-        <inertial>
-            <origin xyz="1.9174124308283903e-17 6.391374769427968e-18 0.011555000000000065" rpy="0 0 0"/>
-            <mass value="0.09427396478246144"/>
-            <inertia ixx="3.3e-05" iyy="3.3e-05" izz="5.8e-05" ixy="0.0" iyz="0.0" ixz="-0.0"/>
-        </inertial>
-        <visual>
-            <origin xyz="-0.0 -0.0 -0.204001" rpy="0 0 0"/>
+            <origin xyz="0.0 0.0 -0.1935" rpy="0 0 0"/>
             <geometry>
             <mesh filename="file://$(find max_description)/meshes/lidar_link.stl" scale="0.001 0.001 0.001"/>
@@ -122,5 +82,5 @@
         </visual>
         <collision>
-            <origin xyz="-0.0 -0.0 -0.204001" rpy="0 0 0"/>
+            <origin xyz="0.0 0.0 -0.1935" rpy="0 0 0"/>
             <geometry>
             <mesh filename="file://$(find max_description)/meshes/lidar_link.stl" scale="0.001 0.001 0.001"/>
@@ -130,10 +90,10 @@
     <link name="camera_link">
         <inertial>
-            <origin xyz="0.014490312898766358 3.7392359944188856e-16 -0.008993541932510896" rpy="0 0 0"/>
-            <mass value="0.23204150441063995"/>
-            <inertia ixx="0.00064" iyy="6e-05" izz="0.000604" ixy="0.0" iyz="-0.0" ixz="0.0"/>
+            <origin xyz="0.013632302340116711 -8.413408858487514e-17 8.326672684688674e-17" rpy="0 0 0"/>
+            <mass value="0.30616096974630597"/>
+            <inertia ixx="0.000806" iyy="9.3e-05" izz="0.000771" ixy="-0.0" iyz="-0.0" ixz="0.0"/>
         </inertial>
         <visual>
-            <origin xyz="-0.1133 -0.0 -0.144" rpy="0 0 0"/>
+            <origin xyz="-0.046567 0.005 -0.0925" rpy="0 0 0"/>
             <geometry>
             <mesh filename="file://$(find max_description)/meshes/camera_link.stl" scale="0.001 0.001 0.001"/>
@@ -142,7 +102,47 @@
         </visual>
         <collision>
-            <origin xyz="-0.1133 -0.0 -0.144" rpy="0 0 0"/>
+            <origin xyz="-0.046567 0.005 -0.0925" rpy="0 0 0"/>
             <geometry>
             <mesh filename="file://$(find max_description)/meshes/camera_link.stl" scale="0.001 0.001 0.001"/>
+            </geometry>
+        </collision>
+    </link>
+    <link name="fr_roller_wheel">
+        <inertial>
+            <origin xyz="1.3877787807814457e-17 6.938893903907228e-18 -5.204170427930421e-18" rpy="0 0 0"/>
+            <mass value="0.01387209506100743"/>
+            <inertia ixx="0.0" iyy="0.0" izz="0.0" ixy="0.0" iyz="0.0" ixz="0.0"/>
+        </inertial>
+        <visual>
+            <origin xyz="-0.07 0.055 -0.0075" rpy="0 0 0"/>
+            <geometry>
+            <mesh filename="file://$(find max_description)/meshes/fr_roller_wheel.stl" scale="0.001 0.001 0.001"/>
+            </geometry>
+            <material name="matte_black"/>
+        </visual>
+        <collision>
+            <origin xyz="-0.07 0.055 -0.0075" rpy="0 0 0"/>
+            <geometry>
+            <mesh filename="file://$(find max_description)/meshes/fr_roller_wheel.stl" scale="0.001 0.001 0.001"/>
+            </geometry>
+        </collision>
+    </link>
+    <link name="fl_roller_wheel">
+        <inertial>
+            <origin xyz="1.3877787807814457e-17 -6.938893903907228e-18 1.9949319973733282e-17" rpy="0 0 0"/>
+            <mass value="0.01387209506100743"/>
+            <inertia ixx="0.0" iyy="0.0" izz="0.0" ixy="0.0" iyz="-0.0" ixz="0.0"/>
+        </inertial>
+        <visual>
+            <origin xyz="-0.07 -0.055 -0.0075" rpy="0 0 0"/>
+            <geometry>
+            <mesh filename="file://$(find max_description)/meshes/fl_roller_wheel.stl" scale="0.001 0.001 0.001"/>
+            </geometry>
+            <material name="matte_black"/>
+        </visual>
+        <collision>
+            <origin xyz="-0.07 -0.055 -0.0075" rpy="0 0 0"/>
+            <geometry>
+            <mesh filename="file://$(find max_description)/meshes/fl_roller_wheel.stl" scale="0.001 0.001 0.001"/>
             </geometry>
         </collision>
@@ -153,38 +153,35 @@
         <origin xyz="0 0 0.0425" rpy="0 0 0"/>
     </joint>
-    <joint name="fl_joint" type="continuous">
-        <origin xyz="0.07309 0.109 0" rpy="0 0 0"/>
+    <joint name="rr_joint" type="continuous">
+        <origin xyz="-0.075 -0.095 0" rpy="0 0 0"/>
         <parent link="base_link"/>
-        <child link="fl_wheel_link"/>
-        <axis xyz="0.0 1.0 0.0"/>
-    </joint>
-    <joint name="fr_joint" type="continuous">
-        <origin xyz="0.07309 -0.109 0" rpy="0 0 0"/>
-        <parent link="base_link"/>
-        <child link="fr_wheel_link"/>
-        <axis xyz="0.0 1.0 0.0"/>
+        <child link="rr_wheel_link"/>
+        <axis xyz="0.0 -1.0 0.0"/>
     </joint>
     <joint name="rl_joint" type="continuous">
-        <origin xyz="-0.0978 0.109 0" rpy="0 0 0"/>
+        <origin xyz="-0.075 0.095 0" rpy="0 0 0"/>
         <parent link="base_link"/>
         <child link="rl_wheel_link"/>
         <axis xyz="0.0 1.0 0.0"/>
     </joint>
-    <joint name="rr_joint" type="continuous">
-        <origin xyz="-0.0978 -0.109 0" rpy="0 0 0"/>
-        <parent link="base_link"/>
-        <child link="rr_wheel_link"/>
-        <axis xyz="0.0 1.0 0.0"/>
-    </joint>
     <joint name="lidar_joint" type="fixed">
-        <origin xyz="0.0 0.0 0.161501" rpy="0 0 0"/>
+        <origin xyz="0.0 0.0 0.151" rpy="0 0 0"/>
         <parent link="base_link"/>
         <child link="lidar_link"/>
-        <axis xyz="0 0 1"/>
     </joint>
     <joint name="camera_joint" type="fixed">
-        <origin xyz="0.1133 0.0 0.1015" rpy="0 0 0"/>
+        <origin xyz="0.046567 -0.005 0.05" rpy="0 0 0"/>
         <parent link="base_link"/>
         <child link="camera_link"/>
     </joint>
+    <joint name="fr_joint" type="fixed">
+        <origin xyz="0.07 -0.055 -0.035" rpy="0 0 0"/>
+        <parent link="base_link"/>
+        <child link="fr_roller_wheel"/>
+    </joint>
+    <joint name="fl_joint" type="fixed">
+        <origin xyz="0.07 0.055 -0.035" rpy="0 0 0"/>
+        <parent link="base_link"/>
+        <child link="fl_roller_wheel"/>
+    </joint>
 </robot>

File: max_description/urdf/trans.xacro (robot description, xacro)
@@ -15,18 +15,4 @@
     </xacro:unless>
   </gazebo>
-  <transmission name="fl_transmission">
-    <plugin>transmission_interface/SimpleTransmission</plugin>
-    <joint name="fl_joint" role="joint_fl">
-      <mechanical_reduction>1.0</mechanical_reduction>
-    </joint>
-    <actuator name="fl_motor" role="actuator_fl"/>
-  </transmission>
-  <transmission name="fr_transmission">
-    <plugin>transmission_interface/SimpleTransmission</plugin>
-    <joint name="fr_joint" role="joint_fr">
-      <mechanical_reduction>1.0</mechanical_reduction>
-    </joint>
-    <actuator name="fr_motor" role="actuator_fr"/>
-  </transmission>
   <transmission name="rl_transmission">
     <plugin>transmission_interface/SimpleTransmission</plugin>
