Commit message: Beginning on diff drive controller

File: max_description/urdf/ros2_control.xacro (robot description, xacro)
@@ -20,20 +20,4 @@
             </hardware>
         </xacro:unless>
-        <joint name="fl_joint">
-            <command_interface name="velocity">
-                <param name="min">-1</param>
-                <param name="max">1</param>
-            </command_interface>
-            <state_interface name="velocity"/>
-            <state_interface name="position"/>
-        </joint>
-        <joint name="fr_joint">
-            <command_interface name="velocity">
-                <param name="min">-1</param>
-                <param name="max">1</param>
-            </command_interface>
-            <state_interface name="velocity"/>
-            <state_interface name="position"/>
-        </joint>
         <joint name="rl_joint">
             <command_interface name="velocity">
