Commit message: urdf basefootprint+baselink

File: max_description/urdf/max.urdf.xacro (robot description, xacro)
@@ -9,5 +9,5 @@
         </inertial>
         <visual>
-            <origin xyz="0 0 0" rpy="0 0 0"/>
+            <origin xyz="0 0 -0.0425" rpy="0 0 0"/>
             <geometry>
             <mesh filename="file://$(find max_description)/meshes/base_link.stl" scale="0.001 0.001 0.001"/>
@@ -22,8 +22,112 @@
         </collision>
     </link>
+    <link name="fl_wheel_link">
+        <inertial>
+            <origin xyz="4.163336342344337e-17 0.010504645034502769 0.0" rpy="0 0 0"/>
+            <mass value="0.16353745126830063"/>
+            <inertia ixx="8.7e-05" iyy="0.000148" izz="8.7e-05" ixy="0.0" iyz="0.0" ixz="0.0"/>
+        </inertial>
+        <visual>
+            <origin xyz="-0.07309 -0.109 -0.0425" rpy="0 0 0"/>
+            <geometry>
+            <mesh filename="file://$(find max_description)/meshes/fl_wheel_link.stl" scale="0.001 0.001 0.001"/>
+            </geometry>
+            <material name="silver"/>
+        </visual>
+        <collision>
+            <origin xyz="-0.07309 -0.109 -0.0425" rpy="0 0 0"/>
+            <geometry>
+            <mesh filename="file://$(find max_description)/meshes/fl_wheel_link.stl" scale="0.001 0.001 0.001"/>
+            </geometry>
+        </collision>
+    </link>
+    <link name="fr_wheel_link">
+        <inertial>
+            <origin xyz="4.163336342344337e-17 -0.01050464503450281 -1.3877787807814457e-17" rpy="0 0 0"/>
+            <mass value="0.16353745126830063"/>
+            <inertia ixx="8.7e-05" iyy="0.000148" izz="8.7e-05" ixy="-0.0" iyz="-0.0" ixz="-0.0"/>
+        </inertial>
+        <visual>
+            <origin xyz="-0.07309 0.109 -0.0425" rpy="0 0 0"/>
+            <geometry>
+            <mesh filename="file://$(find max_description)/meshes/fr_wheel_link.stl" scale="0.001 0.001 0.001"/>
+            </geometry>
+            <material name="silver"/>
+        </visual>
+        <collision>
+            <origin xyz="-0.07309 0.109 -0.0425" rpy="0 0 0"/>
+            <geometry>
+            <mesh filename="file://$(find max_description)/meshes/fr_wheel_link.stl" scale="0.001 0.001 0.001"/>
+            </geometry>
+        </collision>
+    </link>
+    <link name="rl_wheel_link">
+        <inertial>
+            <origin xyz="5.551115123125783e-17 0.010504645034502769 -1.3877787807814457e-17" rpy="0 0 0"/>
+            <mass value="0.16353745126830063"/>
+            <inertia ixx="8.7e-05" iyy="0.000148" izz="8.7e-05" ixy="0.0" iyz="-0.0" ixz="-0.0"/>
+        </inertial>
+        <visual>
+            <origin xyz="0.0978 -0.109 -0.0425" rpy="0 0 0"/>
+            <geometry>
+            <mesh filename="file://$(find max_description)/meshes/rl_wheel_link.stl" scale="0.001 0.001 0.001"/>
+            </geometry>
+            <material name="silver"/>
+        </visual>
+        <collision>
+            <origin xyz="0.0978 -0.109 -0.0425" rpy="0 0 0"/>
+            <geometry>
+            <mesh filename="file://$(find max_description)/meshes/rl_wheel_link.stl" scale="0.001 0.001 0.001"/>
+            </geometry>
+        </collision>
+    </link>
+    <link name="rr_wheel_link">
+        <inertial>
+            <origin xyz="5.551115123125783e-17 -0.01050464503450281 -1.3877787807814457e-17" rpy="0 0 0"/>
+            <mass value="0.16353745126830063"/>
+            <inertia ixx="8.7e-05" iyy="0.000148" izz="8.7e-05" ixy="-0.0" iyz="-0.0" ixz="0.0"/>
+        </inertial>
+        <visual>
+            <origin xyz="0.0978 0.109 -0.0425" rpy="0 0 0"/>
+            <geometry>
+            <mesh filename="file://$(find max_description)/meshes/rr_wheel_link.stl" scale="0.001 0.001 0.001"/>
+            </geometry>
+            <material name="silver"/>
+        </visual>
+        <collision>
+            <origin xyz="0.0978 0.109 -0.0425" rpy="0 0 0"/>
+            <geometry>
+            <mesh filename="file://$(find max_description)/meshes/rr_wheel_link.stl" scale="0.001 0.001 0.001"/>
+            </geometry>
+        </collision>
+    </link>
     <joint name="base_joint" type="fixed">
         <parent link="base_footprint"/>
         <child link="base_link"/>
-        <origin xyz="0 0 0" rpy="0 0 0"/>
+        <origin xyz="0 0 0.0425" rpy="0 0 0"/>
+    </joint>
+    <joint name="fl_joint" type="continuous">
+        <origin xyz="0.07309 0.109 0" rpy="0 0 0"/>
+        <parent link="base_link"/>
+        <child link="fl_wheel_link"/>
+        <axis xyz="0.0 1.0 0.0"/>
+    </joint>
+    <joint name="fr_joint" type="continuous">
+        <origin xyz="0.07309 -0.109 0" rpy="0 0 0"/>
+        <parent link="base_link"/>
+        <child link="fr_wheel_link"/>
+        <axis xyz="0.0 -1.0 0.0"/>
+    </joint>
+    <joint name="rl_joint" type="continuous">
+        <origin xyz="-0.0978 0.109 0" rpy="0 0 0"/>
+        <parent link="base_link"/>
+        <child link="rl_wheel_link"/>
+        <axis xyz="0.0 1.0 0.0"/>
+    </joint>
+    <joint name="rr_joint" type="continuous">
+        <origin xyz="-0.0978 -0.109 0" rpy="0 0 0"/>
+        <parent link="base_link"/>
+        <child link="rr_wheel_link"/>
+        <axis xyz="0.0 -1.0 0.0"/>
     </joint>
 </robot>

Commit message: saving rviz in description package

File: max_description/urdf/max.urdf.xacro (robot description, xacro)
@@ -103,4 +103,24 @@
         </collision>
     </link>
+    <link name="lidar_link">
+        <inertial>
+            <origin xyz="1.9174124308283903e-17 6.391374769427968e-18 0.011555000000000093" rpy="0 0 0"/>
+            <mass value="0.11472963638620308"/>
+            <inertia ixx="4e-05" iyy="4e-05" izz="7e-05" ixy="0.0" iyz="0.0" ixz="-0.0"/>
+        </inertial>
+        <visual>
+            <origin xyz="-0.0 -0.0 -0.204001" rpy="0 0 0"/>
+            <geometry>
+            <mesh filename="file://$(find max_description)/meshes/lidar_link.stl" scale="0.001 0.001 0.001"/>
+            </geometry>
+            <material name="silver"/>
+        </visual>
+        <collision>
+            <origin xyz="-0.0 -0.0 -0.204001" rpy="0 0 0"/>
+            <geometry>
+            <mesh filename="file://$(find max_description)/meshes/lidar_link.stl" scale="0.001 0.001 0.001"/>
+            </geometry>
+        </collision>
+    </link>
     <joint name="base_joint" type="fixed">
         <parent link="base_footprint"/>
@@ -132,3 +152,9 @@
         <axis xyz="0.0 -1.0 0.0"/>
     </joint>
+    <joint name="lidar_joint" type="continuous">
+        <origin xyz="0.0 0.0 0.161501" rpy="0 0 0"/>
+        <parent link="base_link"/>
+        <child link="lidar_link"/>
+        <axis xyz="0 0 1"/>
+    </joint>
 </robot>

Commit message: launch file is complete

File: max_description/urdf/max.urdf.xacro (robot description, xacro)
@@ -2,4 +2,5 @@
 <robot name="max" xmlns:xacro="http://www.ros.org/wiki/xacro">
     <xacro:include filename="$(find max_description)/urdf/materials.xacro" />
+    <xacro:include filename="$(find max_description)/urdf/max.gazebo.xacro" />
     <link name="base_footprint"/>
     <link name="base_link">
@@ -19,5 +20,5 @@
             <origin xyz="0 0 0" rpy="0 0 0"/>
             <geometry>
-            <mesh filename="file://$(find max_description)/meshes/base_link.stl" scale="0.001 0.001 0.001"/>
+                <mesh filename="file://$(find max_description)/meshes/base_link.stl" scale="0.001 0.001 0.001"/>
             </geometry>
         </collision>
@@ -32,5 +33,5 @@
             <origin xyz="-0.07309 -0.109 -0.0425" rpy="0 0 0"/>
             <geometry>
-            <mesh filename="file://$(find max_description)/meshes/fl_wheel_link.stl" scale="0.001 0.001 0.001"/>
+                <mesh filename="file://$(find max_description)/meshes/fl_wheel_link.stl" scale="0.001 0.001 0.001"/>
             </geometry>
             <material name="silver"/>
@@ -39,5 +40,5 @@
             <origin xyz="-0.07309 -0.109 -0.0425" rpy="0 0 0"/>
             <geometry>
-            <mesh filename="file://$(find max_description)/meshes/fl_wheel_link.stl" scale="0.001 0.001 0.001"/>
+                <sphere radius="0.0425"/>
             </geometry>
         </collision>
@@ -59,5 +60,5 @@
             <origin xyz="-0.07309 0.109 -0.0425" rpy="0 0 0"/>
             <geometry>
-            <mesh filename="file://$(find max_description)/meshes/fr_wheel_link.stl" scale="0.001 0.001 0.001"/>
+                <sphere radius="0.0425"/>
             </geometry>
         </collision>
@@ -79,5 +80,5 @@
             <origin xyz="0.0978 -0.109 -0.0425" rpy="0 0 0"/>
             <geometry>
-            <mesh filename="file://$(find max_description)/meshes/rl_wheel_link.stl" scale="0.001 0.001 0.001"/>
+                <sphere radius="0.0425"/>
             </geometry>
         </collision>
@@ -99,5 +100,5 @@
             <origin xyz="0.0978 0.109 -0.0425" rpy="0 0 0"/>
             <geometry>
-            <mesh filename="file://$(find max_description)/meshes/rr_wheel_link.stl" scale="0.001 0.001 0.001"/>
+                <sphere radius="0.0425"/>
             </geometry>
         </collision>
@@ -118,7 +119,4 @@
         <collision>
             <origin xyz="-0.0 -0.0 -0.204001" rpy="0 0 0"/>
-            <geometry>
-            <mesh filename="file://$(find max_description)/meshes/lidar_link.stl" scale="0.001 0.001 0.001"/>
-            </geometry>
         </collision>
     </link>

Commit message: Car is moving--yay

File: max_description/urdf/max.urdf.xacro (robot description, xacro)
@@ -161,5 +161,5 @@
         <parent link="base_link"/>
         <child link="fr_wheel_link"/>
-        <axis xyz="0.0 -1.0 0.0"/>
+        <axis xyz="0.0 1.0 0.0"/>
     </joint>
     <joint name="rl_joint" type="continuous">
@@ -173,5 +173,5 @@
         <parent link="base_link"/>
         <child link="rr_wheel_link"/>
-        <axis xyz="0.0 -1.0 0.0"/>
+        <axis xyz="0.0 1.0 0.0"/>
     </joint>
     <joint name="lidar_joint" type="continuous">

Commit message: Chnaged Lidar Joint continuous to fixed - Lidar simulation failed

File: max_description/urdf/max.urdf.xacro (robot description, xacro)
@@ -175,5 +175,5 @@
         <axis xyz="0.0 1.0 0.0"/>
     </joint>
-    <joint name="lidar_joint" type="continuous">
+    <joint name="lidar_joint" type="fixed">
         <origin xyz="0.0 0.0 0.161501" rpy="0 0 0"/>
         <parent link="base_link"/>

Commit message: wheel stl files changed -: slotted

File: max_description/urdf/max.urdf.xacro (robot description, xacro)
@@ -34,5 +34,5 @@
         </inertial>
         <visual>
-            <origin xyz="-0.07309 -0.109 -0.0425" rpy="0 0 0"/>
+            <origin xyz="-0.35369 -0.109 -0.0425" rpy="0 0 0"/>
             <geometry>
                 <mesh filename="file://$(find max_description)/meshes/fl_wheel_link.stl" scale="0.001 0.001 0.001"/>
@@ -54,5 +54,5 @@
         </inertial>
         <visual>
-            <origin xyz="-0.07309 0.109 -0.0425" rpy="0 0 0"/>
+            <origin xyz="-0.35369 0.109 -0.0425" rpy="0 0 0"/>
             <geometry>
             <mesh filename="file://$(find max_description)/meshes/fr_wheel_link.stl" scale="0.001 0.001 0.001"/>
@@ -74,5 +74,5 @@
         </inertial>
         <visual>
-            <origin xyz="0.0978 -0.109 -0.0425" rpy="0 0 0"/>
+            <origin xyz="-0.1828 -0.109 -0.0425" rpy="0 0 0"/>
             <geometry>
             <mesh filename="file://$(find max_description)/meshes/rl_wheel_link.stl" scale="0.001 0.001 0.001"/>
@@ -94,5 +94,5 @@
         </inertial>
         <visual>
-            <origin xyz="0.0978 0.109 -0.0425" rpy="0 0 0"/>
+            <origin xyz="-0.1828 0.109 -0.0425" rpy="0 0 0"/>
             <geometry>
             <mesh filename="file://$(find max_description)/meshes/rr_wheel_link.stl" scale="0.001 0.001 0.001"/>

Commit message: wheel stl files changed -: slotted

File: max_description/urdf/max.urdf.xacro (robot description, xacro)
@@ -29,7 +29,7 @@
     <link name="fl_wheel_link">
         <inertial>
-            <origin xyz="4.163336342344337e-17 0.010504645034502769 0.0" rpy="0 0 0"/>
-            <mass value="0.16353745126830063"/>
-            <inertia ixx="8.7e-05" iyy="0.000148" izz="8.7e-05" ixy="0.0" iyz="0.0" ixz="0.0"/>
+            <origin xyz="5.551115123125783e-17 -0.010504987657416545 0.0" rpy="0 0 0"/>
+            <mass value="0.15230338417321157"/>
+            <inertia ixx="8.3e-05" iyy="0.000141" izz="8.3e-05" ixy="0.0" iyz="0.0" ixz="0.0"/>
         </inertial>
         <visual>
@@ -41,5 +41,5 @@
         </visual>
         <collision>
-            <origin xyz="-0.07309 -0.109 -0.0425" rpy="0 0 0"/>
+            <origin xyz="-0.35369 -0.109 -0.0425" rpy="0 0 0"/>
             <geometry>
             <mesh filename="file://$(find max_description)/meshes/fl_wheel_link.stl" scale="0.001 0.001 0.001"/>
@@ -49,7 +49,7 @@
     <link name="fr_wheel_link">
         <inertial>
-            <origin xyz="4.163336342344337e-17 -0.01050464503450281 -1.3877787807814457e-17" rpy="0 0 0"/>
-            <mass value="0.16353745126830063"/>
-            <inertia ixx="8.7e-05" iyy="0.000148" izz="8.7e-05" ixy="-0.0" iyz="-0.0" ixz="-0.0"/>
+            <origin xyz="5.551115123125783e-17 0.010504987657416559 0.0" rpy="0 0 0"/>
+            <mass value="0.15230338417321157"/>
+            <inertia ixx="8.3e-05" iyy="0.000141" izz="8.3e-05" ixy="-0.0" iyz="0.0" ixz="0.0"/>
         </inertial>
         <visual>
@@ -61,5 +61,5 @@
         </visual>
         <collision>
-            <origin xyz="-0.07309 0.109 -0.0425" rpy="0 0 0"/>
+            <origin xyz="-0.35369 0.109 -0.0425" rpy="0 0 0"/>
             <geometry>
             <mesh filename="file://$(find max_description)/meshes/fr_wheel_link.stl" scale="0.001 0.001 0.001"/>
@@ -69,7 +69,7 @@
     <link name="rl_wheel_link">
         <inertial>
-            <origin xyz="5.551115123125783e-17 0.010504645034502769 -1.3877787807814457e-17" rpy="0 0 0"/>
-            <mass value="0.16353745126830063"/>
-            <inertia ixx="8.7e-05" iyy="0.000148" izz="8.7e-05" ixy="0.0" iyz="-0.0" ixz="-0.0"/>
+            <origin xyz="1.3877787807814457e-16 0.010504987657416587 0.0" rpy="0 0 0"/>
+            <mass value="0.15230338417321163"/>
+            <inertia ixx="8.3e-05" iyy="0.000141" izz="8.3e-05" ixy="0.0" iyz="0.0" ixz="0.0"/>
         </inertial>
         <visual>
@@ -81,5 +81,5 @@
         </visual>
         <collision>
-            <origin xyz="0.0978 -0.109 -0.0425" rpy="0 0 0"/>
+            <origin xyz="-0.1828 -0.109 -0.0425" rpy="0 0 0"/>
             <geometry>
             <mesh filename="file://$(find max_description)/meshes/rl_wheel_link.stl" scale="0.001 0.001 0.001"/>
@@ -89,7 +89,7 @@
     <link name="rr_wheel_link">
         <inertial>
-            <origin xyz="5.551115123125783e-17 -0.01050464503450281 -1.3877787807814457e-17" rpy="0 0 0"/>
-            <mass value="0.16353745126830063"/>
-            <inertia ixx="8.7e-05" iyy="0.000148" izz="8.7e-05" ixy="-0.0" iyz="-0.0" ixz="0.0"/>
+            <origin xyz="8.326672684688674e-17 -0.010504987657416587 0.0" rpy="0 0 0"/>
+            <mass value="0.15230338417321165"/>
+            <inertia ixx="8.3e-05" iyy="0.000141" izz="8.3e-05" ixy="0.0" iyz="-0.0" ixz="0.0"/>
         </inertial>
         <visual>
@@ -101,5 +101,5 @@
         </visual>
         <collision>
-            <origin xyz="0.0978 0.109 -0.0425" rpy="0 0 0"/>
+            <origin xyz="-0.1828 0.109 -0.0425" rpy="0 0 0"/>
             <geometry>
             <mesh filename="file://$(find max_description)/meshes/rr_wheel_link.stl" scale="0.001 0.001 0.001"/>

Commit message: Descripton update -mass reduction

File: max_description/urdf/max.urdf.xacro (robot description, xacro)
@@ -9,7 +9,7 @@
     <link name="base_link">
         <inertial>
-            <origin xyz="-0.008949251381261427 2.0808612371678153e-17 0.10071250738095076" rpy="0 0 0"/>
-            <mass value="8.307942395442693"/>
-            <inertia ixx="0.041631" iyy="0.061003" izz="0.073974" ixy="-0.0" iyz="-0.0" ixz="0.002477"/>
+            <origin xyz="0.004914987095310725 0.0 0.11525864563546669" rpy="0 0 0"/>
+            <mass value="2.1411582458682883"/>
+            <inertia ixx="0.015376" iyy="0.021164" izz="0.024064" ixy="-0.0" iyz="-0.0" ixz="0.000293"/>
         </inertial>
         <visual>
@@ -29,10 +29,10 @@
     <link name="fl_wheel_link">
         <inertial>
-            <origin xyz="5.551115123125783e-17 -0.010504987657416545 0.0" rpy="0 0 0"/>
+            <origin xyz="4.163336342344337e-17 0.010504987657416559 -1.3877787807814457e-17" rpy="0 0 0"/>
             <mass value="0.15230338417321157"/>
-            <inertia ixx="8.3e-05" iyy="0.000141" izz="8.3e-05" ixy="0.0" iyz="0.0" ixz="0.0"/>
+            <inertia ixx="8.3e-05" iyy="0.000141" izz="8.3e-05" ixy="0.0" iyz="-0.0" ixz="-0.0"/>
         </inertial>
         <visual>
-            <origin xyz="-0.35369 -0.109 -0.0425" rpy="0 0 0"/>
+            <origin xyz="-0.07309 -0.109 -0.0425" rpy="0 0 0"/>
             <geometry>
                 <mesh filename="file://$(find max_description)/meshes/fl_wheel_link.stl" scale="0.001 0.001 0.001"/>
@@ -41,5 +41,5 @@
         </visual>
         <collision>
-            <origin xyz="-0.35369 -0.109 -0.0425" rpy="0 0 0"/>
+            <origin xyz="-0.07309 -0.109 -0.0425" rpy="0 0 0"/>
             <geometry>
             <mesh filename="file://$(find max_description)/meshes/fl_wheel_link.stl" scale="0.001 0.001 0.001"/>
@@ -49,10 +49,10 @@
     <link name="fr_wheel_link">
         <inertial>
-            <origin xyz="5.551115123125783e-17 0.010504987657416559 0.0" rpy="0 0 0"/>
+            <origin xyz="4.163336342344337e-17 -0.010504987657416545 -1.3877787807814457e-17" rpy="0 0 0"/>
             <mass value="0.15230338417321157"/>
-            <inertia ixx="8.3e-05" iyy="0.000141" izz="8.3e-05" ixy="-0.0" iyz="0.0" ixz="0.0"/>
+            <inertia ixx="8.3e-05" iyy="0.000141" izz="8.3e-05" ixy="0.0" iyz="0.0" ixz="-0.0"/>
         </inertial>
         <visual>
-            <origin xyz="-0.35369 0.109 -0.0425" rpy="0 0 0"/>
+            <origin xyz="-0.07309 0.109 -0.0425" rpy="0 0 0"/>
             <geometry>
             <mesh filename="file://$(find max_description)/meshes/fr_wheel_link.stl" scale="0.001 0.001 0.001"/>
@@ -61,5 +61,5 @@
         </visual>
         <collision>
-            <origin xyz="-0.35369 0.109 -0.0425" rpy="0 0 0"/>
+            <origin xyz="-0.07309 0.109 -0.0425" rpy="0 0 0"/>
             <geometry>
             <mesh filename="file://$(find max_description)/meshes/fr_wheel_link.stl" scale="0.001 0.001 0.001"/>
@@ -69,10 +69,10 @@
     <link name="rl_wheel_link">
         <inertial>
-            <origin xyz="1.3877787807814457e-16 0.010504987657416587 0.0" rpy="0 0 0"/>
+            <origin xyz="6.938893903907228e-17 0.010504987657416559 0.0" rpy="0 0 0"/>
             <mass value="0.15230338417321163"/>
-            <inertia ixx="8.3e-05" iyy="0.000141" izz="8.3e-05" ixy="0.0" iyz="0.0" ixz="0.0"/>
+            <inertia ixx="8.3e-05" iyy="0.000141" izz="8.3e-05" ixy="0.0" iyz="-0.0" ixz="0.0"/>
         </inertial>
         <visual>
-            <origin xyz="-0.1828 -0.109 -0.0425" rpy="0 0 0"/>
+            <origin xyz="0.0978 -0.109 -0.0425" rpy="0 0 0"/>
             <geometry>
             <mesh filename="file://$(find max_description)/meshes/rl_wheel_link.stl" scale="0.001 0.001 0.001"/>
@@ -81,5 +81,5 @@
         </visual>
         <collision>
-            <origin xyz="-0.1828 -0.109 -0.0425" rpy="0 0 0"/>
+            <origin xyz="0.0978 -0.109 -0.0425" rpy="0 0 0"/>
             <geometry>
             <mesh filename="file://$(find max_description)/meshes/rl_wheel_link.stl" scale="0.001 0.001 0.001"/>
@@ -89,10 +89,10 @@
     <link name="rr_wheel_link">
         <inertial>
-            <origin xyz="8.326672684688674e-17 -0.010504987657416587 0.0" rpy="0 0 0"/>
-            <mass value="0.15230338417321165"/>
-            <inertia ixx="8.3e-05" iyy="0.000141" izz="8.3e-05" ixy="0.0" iyz="-0.0" ixz="0.0"/>
+            <origin xyz="6.938893903907228e-17 -0.010504987657416559 -2.0816681711721685e-17" rpy="0 0 0"/>
+            <mass value="0.15230338417321163"/>
+            <inertia ixx="8.3e-05" iyy="0.000141" izz="8.3e-05" ixy="-0.0" iyz="0.0" ixz="0.0"/>
         </inertial>
         <visual>
-            <origin xyz="-0.1828 0.109 -0.0425" rpy="0 0 0"/>
+            <origin xyz="0.0978 0.109 -0.0425" rpy="0 0 0"/>
             <geometry>
             <mesh filename="file://$(find max_description)/meshes/rr_wheel_link.stl" scale="0.001 0.001 0.001"/>
@@ -101,5 +101,5 @@
         </visual>
         <collision>
-            <origin xyz="-0.1828 0.109 -0.0425" rpy="0 0 0"/>
+            <origin xyz="0.0978 0.109 -0.0425" rpy="0 0 0"/>
             <geometry>
             <mesh filename="file://$(find max_description)/meshes/rr_wheel_link.stl" scale="0.001 0.001 0.001"/>
@@ -109,7 +109,7 @@
     <link name="lidar_link">
         <inertial>
-            <origin xyz="1.9174124308283903e-17 6.391374769427968e-18 0.011555000000000093" rpy="0 0 0"/>
-            <mass value="0.11472963638620308"/>
-            <inertia ixx="4e-05" iyy="4e-05" izz="7e-05" ixy="0.0" iyz="0.0" ixz="-0.0"/>
+            <origin xyz="1.9174124308283903e-17 6.391374769427968e-18 0.011555000000000065" rpy="0 0 0"/>
+            <mass value="0.09427396478246144"/>
+            <inertia ixx="3.3e-05" iyy="3.3e-05" izz="5.8e-05" ixy="0.0" iyz="0.0" ixz="-0.0"/>
         </inertial>
         <visual>
@@ -130,6 +130,6 @@
         <inertial>
             <origin xyz="0.014490312898766358 3.7392359944188856e-16 -0.008993541932510896" rpy="0 0 0"/>
-            <mass value="1.7184205751165316"/>
-            <inertia ixx="0.00474" iyy="0.000448" izz="0.004472" ixy="0.0" iyz="-0.0" ixz="0.0"/>
+            <mass value="0.23204150441063995"/>
+            <inertia ixx="0.00064" iyy="6e-05" izz="0.000604" ixy="0.0" iyz="-0.0" ixz="0.0"/>
         </inertial>
         <visual>

Commit message: fixed -1 in urdf, wheel going oppoiste

File: max_description/urdf/max.urdf.xacro (robot description, xacro)
@@ -157,5 +157,5 @@
         <parent link="base_link"/>
         <child link="rr_wheel_link"/>
-        <axis xyz="0.0 -1.0 0.0"/>
+        <axis xyz="0.0 1.0 0.0"/>
     </joint>
     <joint name="rl_joint" type="continuous">
